Commit message: Basic sim working

File: s_description/urdf/gazebo.urdf.xacro (robot description, xacro)
@@ -1,114 +1,4 @@
 <?xml version="1.0"?>
 <robot xmlns:xacro="http://ros.org/wiki/xacro">
-  <xacro:macro name="RealsenseGazebo" params="cam_name">
-    <!-- depth cam -->
-    <gazebo reference="${cam_name}_link">
-      <material>Gazebo/Black</material>
-    </gazebo>
-    <gazebo reference="${cam_name}_color_frame" />
-    <gazebo reference="${cam_name}_color_optical_frame" />
-    <gazebo reference="${cam_name}_depth_frame" />
-    <gazebo reference="${cam_name}_depth_optical_frame" />
-    <gazebo reference="${cam_name}_joint" />
-    <gazebo reference="${cam_name}_color_joint" />
-    <gazebo reference="${cam_name}_depth_joint" />
-    <gazebo reference="${cam_name}_color_optical_joint" />
-    <gazebo reference="${cam_name}_depth_optical_joint" />
-    <!-- generate the RGB camera image -->
-    <gazebo reference="cam_rgb_frame">
-      <sensor name="cam_rgb" type="camera">
-        <always_on>true</always_on>
-        <visualize>true</visualize>
-        <update_rate>15</update_rate>
-        <camera name="cam_rgb">
-          <horizontal_fov>1.085595</horizontal_fov>
-          <image>
-            <width>1280</width>
-            <height>960</height>
-            <format>RGB8</format>
-          </image>
-          <clip>
-            <near>0.03</near>
-            <far>1000</far>
-          </clip>
-          <noise>
-            <type>gaussian</type>
-            <!-- Noise is sampled independently per pixel on each frame.
-                        That pixel's noise value is added to each of its color
-                        channels, which at that point lie in the range [0,1]. -->
-            <mean>0.0</mean>
-            <stddev>0.007</stddev>
-          </noise>
-        </camera>
-        <plugin name="cam_rgb_driver" filename="libgazebo_ros_camera.so">
-          <ros>
-            <!-- <namespace></namespace> -->
-            <!--
-                    <remapping>${cam_name}/image_raw:=cam_rgb/image_raw</remapping>
-                    <remapping>${cam_name}/image_raw/compressed:=${cam_name}/color/image_raw/compressed</remapping>
-                    <remapping>${cam_name}/image_raw/theora:=${cam_name}/color/image_raw/theora</remapping>
-            <remapping>${cam_name}/image_raw/compressedDepth:=${cam_name}/color/image_raw/compressedDepth</remapping>
-                    <remapping>${cam_name}/camera_info:=${cam_name}/color/camera_info</remapping>
-                    -->
-          </ros>
-          <!-- Set camera name. If empty, defaults to sensor name (i.e. "sensor_name") -->
-          <camera_name>cam_rgb</camera_name>
-          <!-- camera_name>omit so it defaults to sensor name</camera_name-->
-          <frame_name>cam_rgb_frame</frame_name>
-        </plugin>
-      </sensor>
-    </gazebo>
-    <!--  Add an RGBD camera -->
-    <gazebo reference="${cam_name}_link">
-      <sensor name="${cam_name}" type="depth">
-        <always_on>true</always_on>
-        <visualize>true</visualize>
-        <update_rate>15</update_rate>
-        <camera name="${cam_name}">
-          <horizontal_fov>1.085595</horizontal_fov>
-          <image>
-            <width>640</width>
-            <height>480</height>
-            <format>Z16</format>
-          </image>
-          <clip>
-            <near>0.04</near>
-            <far>2.0</far>
-          </clip>
-          <noise>
-            <type>gaussian</type>
-            <!-- Noise is sampled independently per pixel on each frame.
-                            That pixel's noise value is added to each of its color
-                            channels, which at that point lie in the range [0,1]. -->
-            <mean>0.0</mean>
-            <stddev>0.07</stddev>
-          </noise>
-        </camera>
-        <plugin name="${cam_name}_driver" filename="libgazebo_ros_camera.so">
-          <ros>
-            <remapping>${cam_name}/image_raw:=${cam_name}/color/image_raw</remapping>
-            <remapping>${cam_name}/image_raw/compressed:=${cam_name}/color/image_raw/compressed</remapping>
-            <remapping>${cam_name}/image_raw/theora:=${cam_name}/color/image_raw/theora</remapping>
-            <remapping>
-              ${cam_name}/image_raw/compressedDepth:=${cam_name}/color/image_raw/compressedDepth</remapping>
-            <remapping>${cam_name}/camera_info:=${cam_name}/color/camera_info</remapping>
-            <remapping>${cam_name}/depth/image_raw:=${cam_name}/depth/image_rect_raw</remapping>
-            <remapping>
-              ${cam_name}/depth/image_raw/compressed:=${cam_name}/depth/image_rect_raw/compressed</remapping>
-            <remapping>${cam_name}/depth/image_raw/theora:=${cam_name}/depth/image_rect_raw/theora</remapping>
-            <remapping>
-              ${cam_name}/depth/image_raw/compressedDepth:=${cam_name}/depth/image_rect_raw/compressedDepth</remapping>
-            <!-- remapping>${cam_name}/camera_info_depth:=${cam_name}/depth/camera_info</remapping -->
-            <remapping>${cam_name}/points:=${cam_name}/depth/color/points</remapping>
-          </ros>
-          <camera_name>${cam_name}</camera_name>
-          <frame_name>${cam_name}_depth_optical_frame</frame_name>
-          <hack_baseline>0.07</hack_baseline>
-          <min_depth>0.4</min_depth>
-          <max_depth>2.0</max_depth>
-        </plugin>
-      </sensor>
-    </gazebo>
-  </xacro:macro>
   <!-- This first link called "world" is empty -->
   <!-- <link name="world"></link> -->
