Commit message: Sim through navigation working better. Next up, slam.

File: s_description/urdf/ld06.urdf.xacro (robot description, xacro)
@@ -138,4 +138,8 @@
     <gazebo reference="lidar_frame_${lidar_prefix}">
       <sensor name="sensor_ray_${lidar_prefix}" type="ray">
+        <always_on>true</always_on>
+        <update_rate>10</update_rate>
+        <pose>0 0 0 0 0 0</pose>
+        <visualize>true</visualize>
         <ray>
           <scan>
@@ -148,23 +152,23 @@
           </scan>
           <range>
-            <min>0.05</min>
+            <min>0.08</min>
             <max>10.0</max>
           </range>
-          <noise>
+          <!-- <noise>
             <type>gaussian</type>
             <mean>0.0</mean>
             <stddev>0.02</stddev>
-          </noise>
+          </noise> -->
         </ray>
-        <always_on>true</always_on>
-        <update_rate>10.0</update_rate>
         <plugin name="laserscan_${lidar_prefix}" filename="libgazebo_ros_ray_sensor.so">
           <ros>
             <remapping>~/out:=/scan_${lidar_prefix}</remapping>
           </ros>
+          <always_on>true</always_on>
+          <frame_name>lidar_frame_${lidar_prefix}</frame_name>
           <output_type>sensor_msgs/LaserScan</output_type>
-          <frame_name>lidar_frame_${lidar_prefix}</frame_name>
+          <topic_name>/scan_${lidar_prefix}</topic_name>
+          <update_rate>10.0</update_rate>
         </plugin>
-        <visualize>1</visualize>
       </sensor>
       <material>

File: s_description/urdf/material.urdf.xacro (robot description, xacro)
@@ -19,4 +19,9 @@
 -->
 <robot xmlns:xacro="http://ros.org/wiki/xacro" name="material">
+    <gazebo reference="base_link">
+        <material>
+            <color rgba="0.516 0.527 0.535 1" />
+        </material>
+    </gazebo>
     <material name="aluminum_frame">
         <color rgba="0.516 0.527 0.535 1" />
