Commit message: Moved aluminum_frame material to base urdf

File: s_description/urdf/material.urdf.xacro (robot description, xacro)
@@ -19,9 +19,4 @@
 -->
 <robot xmlns:xacro="http://ros.org/wiki/xacro" name="material">
-    <gazebo reference="base_link">
-        <material>
-            <color rgba="0.516 0.527 0.535 1" />
-        </material>
-    </gazebo>
     <material name="aluminum_frame">
         <color rgba="0.516 0.527 0.535 1" />
