Commit message: Added description and rviz

File: s_description/urdf/base.urdf.xacro (robot description, xacro)
@@ -18,14 +18,14 @@
 SOFTWARE.
 -->
-<robot xmlns:xacro="http://ros.org/wiki/xacro" name="ravel">
-    <xacro:include filename="$(find raven_description)/urdf/raven_properties.urdf.xacro" />
-    <xacro:include filename="$(find raven_description)/urdf/caster.urdf.xacro" />
-    <xacro:include filename="$(find raven_description)/urdf/depthai_macro.urdf.xacro" />
-    <xacro:include filename="$(find raven_description)/urdf/inertials.xacro" />
-    <xacro:include filename="$(find raven_description)/urdf/ld06.urdf.xacro" />
-    <xacro:include filename="$(find raven_description)/urdf/material.urdf.xacro" />
-    <xacro:include filename="$(find raven_description)/urdf/raven_gazebo.urdf.xacro" />
-    <xacro:include filename="$(find raven_description)/urdf/wheel.urdf.xacro" />
-    <xacro:include filename="$(find raven_description)/urdf/oakd.urdf.xacro" />
+<robot xmlns:xacro="http://ros.org/wiki/xacro" name="base">
+    <xacro:include filename="$(find s_description)/urdf/properties.urdf.xacro" />
+    <xacro:include filename="$(find s_description)/urdf/caster.urdf.xacro" />
+    <xacro:include filename="$(find s_description)/urdf/depthai_macro.urdf.xacro" />
+    <xacro:include filename="$(find s_description)/urdf/inertials.xacro" />
+    <xacro:include filename="$(find s_description)/urdf/ld06.urdf.xacro" />
+    <xacro:include filename="$(find s_description)/urdf/material.urdf.xacro" />
+    <xacro:include filename="$(find s_description)/urdf/gazebo.urdf.xacro" />
+    <xacro:include filename="$(find s_description)/urdf/wheel.urdf.xacro" />
+    <xacro:include filename="$(find s_description)/urdf/oakd.urdf.xacro" />
     <link name="base_link">
         <collision>
@@ -99,39 +99,6 @@
         <origin xyz="${(body_length / 2) + 0.030}  ${((body_width / 2) - 0.0)} 0.040" rpy="0 0 0" />
     </xacro:ld06>
-    <!-- T265 y tilt is 31 degrees or 0.541 radians -->
-    <!-- Visual odometry camera -->
-    <!-- <link name="t265_pose_frame">
-        <collision>
-            <geometry>
-                <box size="${t265_width} ${t265_length} ${t265_height}" />
-                <origin xyz="0 0 0" rpy="0.0 0.0 0.0" />
-            </geometry>
-        </collision>
-        <visual>
-            <geometry>
-                <box size="${t265_width} ${t265_length} ${t265_height}" />
-            </geometry>
-            <origin xyz="0 0 0" rpy="0.0 0.0 0.0" />
-            <material name="t265_material" />
-        </visual>
-    </link>
-    <gazebo reference="t265_pose_frame">
-        <material>
-            Gazebo/DarkGrey
-        </material>
-    </gazebo>
-    <joint name="t265_to_base_footprint" type="fixed">
-        <parent link="t265_rotate_frame" />
-        <child link="base_footprint" />
-        <origin xyz="-${t265_x_offset} 0 -${t265_z_offset}" rpy="0 0 0" />
-    </joint>
-    <link name="t265_rotate_frame" />
-    <joint name="t265_rotator_joint" type="fixed">
-        <parent link="t265_pose_frame" />
-        <child link="t265_rotate_frame" />
-        <origin xyz="0 0 0" rpy="0 0 0" />
-    </joint> -->
-    <xacro:include filename="$(find raven_description)/urdf/time_of_flight.urdf.xacro" />
-    <xacro:include filename="$(find raven_description)/urdf/sonar.urdf.xacro" />
+    <xacro:include filename="$(find s_description)/urdf/time_of_flight.urdf.xacro" />
+    <xacro:include filename="$(find s_description)/urdf/sonar.urdf.xacro" />
     <!-- <xacro:depthai_camera
         camera_name="oakd_left"

File: s_description/urdf/oakd.urdf.xacro (robot description, xacro)
@@ -17,5 +17,5 @@
         <geometry>
           <!-- <box size="${oakd_length} ${oakd_width} ${oakd_depth}" /> -->
-          <mesh filename="file://$(find raven_description)/meshes/OAK-D.dae" />
+          <mesh filename="file://$(find s_description)/meshes/OAK-D.dae" />
         </geometry>
         <color rgba="0.15 0.15 0.15 1" />

Commit message: Basic sim/real launches work. See TODO for issues.

File: s_description/urdf/base.urdf.xacro (robot description, xacro)
@@ -61,14 +61,4 @@
     </gazebo>
     <link name="base_footprint" />
-    <!--joint name="odom_to_odom_frame_joint" type="fixed">
-        <origin xyz="0 0 0" rpy="0 0 0" />
-        <parent link="odom" />
-        <child link="odom_frame" />
-    </joint> -->
-    <!-- joint name="odom_frame_to_t265_pose_frame_joint" type="fixed">
-        <origin xyz="0 0 0" rpy="0 0 0" />> <parent link="odom_frame" />
-        <child
-            link="t265_pose_frame" />
-    </joint> -->
     <joint name="base_footprint_joint" type="fixed">
         <origin xyz="0 0 ${base_to_floor_z_offset}" rpy="0 0 0" />

File: s_description/urdf/gazebo.urdf.xacro (robot description, xacro)
@@ -13,5 +13,5 @@
     <plugin name="differential_drive_controller" filename="libgazebo_ros_diff_drive.so">
       <ros>
-        <!-- <argument>odom:=odom_unfiltered</argument> -->
+        <argument>odom:=odom/unfiltered</argument>
       </ros>
       <updateRate>100</updateRate>
@@ -23,5 +23,5 @@
       <robot_base_frame>base_footprint</robot_base_frame>
       <publish_odom>true</publish_odom>
-      <publish_odom_tf>true</publish_odom_tf>
+      <publish_odom_tf>false</publish_odom_tf>
       <publish_wheel_tf>true</publish_wheel_tf>
       <odometry_frame>odom</odometry_frame>

Commit message: More or less have the launch files working. Simulation is still jittery.

File: s_description/urdf/base.urdf.xacro (robot description, xacro)
@@ -91,4 +91,8 @@
     <xacro:include filename="$(find s_description)/urdf/time_of_flight.urdf.xacro" />
     <xacro:include filename="$(find s_description)/urdf/sonar.urdf.xacro" />
+    <xacro:diff_drive_controller
+        wheel_separation="${body_width * (2 * wheel_center_offset)}"
+        wheel_radius="${wheel_radius}"
+    />
     <!-- <xacro:depthai_camera
         camera_name="oakd_left"

File: s_description/urdf/gazebo.urdf.xacro (robot description, xacro)
@@ -1,30 +1,22 @@
-<?xml version="1.0"?>
 <robot xmlns:xacro="http://ros.org/wiki/xacro">
-  <!-- This first link called "world" is empty -->
-  <!-- <link name="world"></link> -->
-  <!-- A simple fixed joint from our empty world link, to our base. -->
-  <!-- The base origin is offset from the world origin. -->
-  <!-- <joint name="base_joint" type="fixed">
-    <origin xyz="0 0 0" rpy="0 -0.541 0" />
-    <parent link="world" />
-    <child link="odom" />
-  </joint> -->
-  <gazebo>
-    <plugin name="differential_drive_controller" filename="libgazebo_ros_diff_drive.so">
-      <ros>
-        <argument>odom:=odom/unfiltered</argument>
-      </ros>
-      <updateRate>100</updateRate>
-      <left_joint>front_left_wheel_joint</left_joint>
-      <right_joint>front_right_wheel_joint</right_joint>
-      <wheel_separation>${body_width * (2 * wheel_center_offset)}</wheel_separation>
-      <wheel_diameter>${wheel_radius * 2}</wheel_diameter>
-      <max_wheel_acceleration>1.0</max_wheel_acceleration>
-      <robot_base_frame>base_footprint</robot_base_frame>
-      <publish_odom>true</publish_odom>
-      <publish_odom_tf>false</publish_odom_tf>
-      <publish_wheel_tf>true</publish_wheel_tf>
-      <odometry_frame>odom</odometry_frame>
-  </plugin>
-  </gazebo>
+  <xacro:macro name="diff_drive_controller" params="wheel_separation wheel_radius">
+    <gazebo>
+      <plugin name="differential_drive_controller" filename="libgazebo_ros_diff_drive.so">
+        <ros>
+          <argument>odom:=odom/unfiltered</argument>
+        </ros>
+        <updateRate>100</updateRate>
+        <left_joint>front_left_wheel_joint</left_joint>
+        <right_joint>front_right_wheel_joint</right_joint>
+        <wheel_separation>${wheel_separation}</wheel_separation>
+        <wheel_diameter>${wheel_radius * 2}</wheel_diameter>
+        <max_wheel_acceleration>1.0</max_wheel_acceleration>
+        <robot_base_frame>base_footprint</robot_base_frame>
+        <publish_odom>true</publish_odom>
+        <publish_odom_tf>false</publish_odom_tf>
+        <publish_wheel_tf>true</publish_wheel_tf>
+        <odometry_frame>odom</odometry_frame>
+      </plugin>
+    </gazebo>
+  </xacro:macro>
 </robot>

Commit message: Fix aluminum_frame material for gazebo

File: s_description/urdf/base.urdf.xacro (robot description, xacro)
@@ -54,8 +54,7 @@
         </inertial>
     </link>
-    <gazebo
-        reference="base_link">
-        <material>
-            aluminum_frame
+    <gazebo reference="base_link">
+        <material name="aluminum_frame">
+            <color rgba="0.516 0.527 0.535 1" />
         </material>
     </gazebo>

Commit message: Simulation finally working. Need to turn on two lasers.

File: s_description/urdf/base.urdf.xacro (robot description, xacro)
@@ -65,31 +65,41 @@
         <child link="base_link" />
     </joint>
-    <xacro:wheel wheel_prefix="front_left">
-        <origin xyz="0 ${(body_width/2)+wheel_center_offset} -${gear_box_center_height}" rpy="0 0 0" />
-    </xacro:wheel>
-    <xacro:wheel wheel_prefix="front_right">
-        <origin xyz="0 -${(body_width/2)+wheel_center_offset} -${gear_box_center_height}"
-            rpy="0 0 0" />
-    </xacro:wheel>
-    <xacro:caster wheel_prefix="fcaster">
-        <origin xyz="${fwheel_offset} 0.0 -${wheel_radius + gear_box_center_height - caster_radius}"
-            rpy="0 0 0" />
-    </xacro:caster>
-    <xacro:caster wheel_prefix="rcaster">
-        <origin
-            xyz="${-fwheel_offset} 0.0 -${wheel_radius + gear_box_center_height - caster_radius}"
-            rpy="0 0 0" />
-    </xacro:caster>
+    <xacro:wheel
+        side="left"
+        radius="${wheel_radius}"
+        width="${wheel_width}"
+        pos_x="${wheel_pos_x}"
+        pos_y="${wheel_pos_y}"
+        pos_z="${wheel_pos_z}"
+        mass="${wheel_mass}"
+    />
+    <xacro:wheel
+        side="right"
+        radius="${wheel_radius}"
+        width="${wheel_width}"
+        pos_x="${wheel_pos_x}"
+        pos_y="${-wheel_pos_y}"
+        pos_z="${wheel_pos_z}"
+        mass="${wheel_mass}"
+    />
+    <xacro:caster_wheel
+        side="front"
+        mass="0.01"
+    />
+    <xacro:caster_wheel
+        side="rear"
+        mass="0.01"
+    />
     <xacro:ld06 lidar_prefix="right_rear">
-        <origin xyz="${-(body_length / 2) - 0.030}  -${((body_width / 2) - 0)} 0.200"
+        <origin xyz="0 0  0.400"
             rpy="0 0 ${M_PI}" />
     </xacro:ld06>
-    <xacro:ld06 lidar_prefix="left_front">
+    <!-- <xacro:ld06 lidar_prefix="left_front">
         <origin xyz="${(body_length / 2) + 0.030}  ${((body_width / 2) - 0.0)} 0.040" rpy="0 0 0" />
-    </xacro:ld06>
+    </xacro:ld06> -->
     <xacro:include filename="$(find s_description)/urdf/time_of_flight.urdf.xacro" />
     <xacro:include filename="$(find s_description)/urdf/sonar.urdf.xacro" />
     <xacro:diff_drive_controller
-        wheel_separation="${body_width * (2 * wheel_center_offset)}"
+        wheel_separation="${wheel_pos_y * 2}"
         wheel_radius="${wheel_radius}"
     />

File: s_description/urdf/caster.urdf.xacro (robot description, xacro)
@@ -18,36 +18,50 @@
 SOFTWARE.
 -->
-<robot xmlns:xacro="http://ros.org/wiki/xacro" name="caster">
-	<xacro:macro name="caster" params="wheel_prefix *joint_pose">
-		<link name="${wheel_prefix}_wheel_link">
+<robot xmlns:xacro="http://ros.org/wiki/xacro">
+	<xacro:macro name="caster_wheel" params="side mass">
+		<xacro:property name="caster_wheel_radius" value="0.0381" />
+		<xacro:if value="${side == 'front'}">
+			<xacro:property name="caster_wheel_x" value="${fwheel_offset}" />
+		</xacro:if>
+		<xacro:if value="${side == 'rear'}">
+			<xacro:property name="caster_wheel_x" value="${-fwheel_offset}" />
+		</xacro:if>
+		<link name="${side}_caster_wheel_link">
+			<visual>
+				<origin xyz="0 0 0" rpy="0 0 0" />
+				<geometry>
+					<sphere radius="${caster_wheel_radius}" />
+				</geometry>
+				<material name="red">
+					<color rgba="0.416 0.051 0.047 1.0" />
+				</material>
+			</visual>
 			<collision>
-				<origin xyz="0 0 0" rpy="${M_PI/2} 0 0" />
+				<origin xyz="0 0 0" rpy="0 0 0" />
 				<geometry>
-					<cylinder length="${caster_width}" radius="${caster_radius}" />
+					<sphere radius="${caster_wheel_radius}" />
 				</geometry>
 			</collision>
 			<inertial>
-				<mass value="0.01" />
-				<origin xyz="0 0 0" />
-				<inertia ixx="0.02467" ixy="0" ixz="0" iyy="0.04411" iyz="0" izz="0.02467" />
+				<origin xyz="0 0 0" rpy="0 0 0" />
+				<mass value="${mass}" />
+				<inertia ixx="${(2/5) * mass * (caster_wheel_radius * caster_wheel_radius)}" ixy="0"
+					ixz="0"
+					iyy="${(2/5) * mass * (caster_wheel_radius * caster_wheel_radius)}" iyz="0"
+					izz="${(2/5) * mass * (caster_wheel_radius * caster_wheel_radius)}" />
 			</inertial>
-			<visual>
-				<geometry>
-					<cylinder length="${caster_width}" radius="${caster_radius}" />
-				</geometry>
-				<material name="caster_wheel_material" />
-				<origin xyz="0 0 0" rpy="${M_PI/2} 0 0" />
-			</visual>
 		</link>
-		<joint name="${wheel_prefix}_wheel" type="fixed">
-			<parent link="base_link" />
-			<child link="${wheel_prefix}_wheel_link" />
-			<xacro:insert_block name="joint_pose" />
-		</joint>
-		<gazebo reference="${wheel_prefix}_wheel_link">
-			<mu1>0.00001</mu1>
-			<mu2>0.00001</mu2>
+		<gazebo reference="${side}_caster_wheel_link">
+			<mu1>0.01</mu1>
+			<mu2>0.01</mu2>
 			<material>Gazebo/Red</material>
 		</gazebo>
+		<joint name="${side}_caster_wheel_joint" type="fixed">
+			<parent link="base_link" />
+			<child link="${side}_caster_wheel_link" />
+			<origin
+				xyz="${caster_wheel_x} 0 -${wheel_radius + gear_box_center_height - caster_wheel_radius}"
+				rpy="0 0 0" />
+		</joint>
 	</xacro:macro>
 </robot>

File: s_description/urdf/gazebo.urdf.xacro (robot description, xacro)
@@ -7,6 +7,6 @@
         </ros>
         <updateRate>100</updateRate>
-        <left_joint>front_left_wheel_joint</left_joint>
-        <right_joint>front_right_wheel_joint</right_joint>
+        <left_joint>left_wheel_joint</left_joint>
+        <right_joint>right_wheel_joint</right_joint>
         <wheel_separation>${wheel_separation}</wheel_separation>
         <wheel_diameter>${wheel_radius * 2}</wheel_diameter>

File: s_description/urdf/ld06.urdf.xacro (robot description, xacro)
@@ -152,6 +152,7 @@
           </scan>
           <range>
-            <min>0.08</min>
+            <min>0.1</min>
             <max>10.0</max>
+            <resolution>0.01</resolution>
           </range>
           <!-- <noise>
@@ -163,5 +164,5 @@
         <plugin name="laserscan_${lidar_prefix}" filename="libgazebo_ros_ray_sensor.so">
           <ros>
-            <remapping>~/out:=/scan_${lidar_prefix}</remapping>
+            <remapping>~/out:=/scan</remapping>
           </ros>
           <always_on>true</always_on>

File: s_description/urdf/properties.urdf.xacro (robot description, xacro)
@@ -16,4 +16,8 @@
   <xacro:property name="wheel_radius" value="0.10" />
   <xacro:property name="wheel_center_offset" value="0.030" />
+  <xacro:property name="wheel_mass" value=".1" />
+  <xacro:property name="wheel_pos_x" value="0.0" />
+  <xacro:property name="wheel_pos_y" value="${(body_width/2)+wheel_center_offset}" />
+  <xacro:property name="wheel_pos_z" value="-${gear_box_center_height}" />
   <xacro:property name="wheel_width" value="0.0254" />
   <xacro:property name="base_to_floor_z_offset" value="${wheel_radius+gear_box_center_height}" />

File: s_description/urdf/wheel.urdf.xacro (robot description, xacro)
@@ -18,47 +18,44 @@
 SOFTWARE.
 -->
-<robot xmlns:xacro="http://ros.org/wiki/xacro" name="wheel">
-	<xacro:macro name="wheel" params="wheel_prefix *joint_pose">
-		<link name="${wheel_prefix}_wheel_link">
-			<collision>
-				<origin xyz="0 0 0" rpy="${M_PI/2} 0 0" />
-				<geometry>
-					<cylinder length="${wheel_width}" radius="${wheel_radius}" />
-				</geometry>
-			</collision>
-			<inertial>
-				<mass value="2.637" />
-				<origin xyz="0 0 0" />
-				<inertia ixx="0.02467" ixy="0" ixz="0" iyy="0.04411" iyz="0" izz="0.02467" />
-			</inertial>
-			<visual>
-				<origin xyz="0 0 0" rpy="${M_PI/2} 0 0" />
-				<geometry>
-					<cylinder length="${wheel_width}" radius="${wheel_radius}" />
-				</geometry>
-				<material name="wheel_material" />
-			</visual>
-		</link>
-		<joint name="${wheel_prefix}_wheel_joint" type="continuous">
-			<parent link="base_link" />
-			<child link="${wheel_prefix}_wheel_link" />
-			<xacro:insert_block name="joint_pose" />
-			<axis xyz="0 1 0" rpy="0 0 0" />
-			<limit effort="100" velocity="3" />
-			<dynamics damping="0.1" friction="0.5" />
-		</joint>
-		<gazebo reference="${wheel_prefix}_wheel_link">
-			<mu1 value="10000.0" />
-			<mu2 value="10000.0" />
-			<kp value="1e13" />
-			<kd value="1" />
-			<!-- <mu1>200.0</mu1>
-			<mu2>100.0</mu2>
-			<kp>1000000.0</kp>
-			<kd>1.0</kd>
-			<max_vel>0.01</max_vel>
-			<min_depth>0.001</min_depth> -->
-			<material>Gazebo/Black</material>
-		</gazebo>
-	</xacro:macro>
+<robot xmlns:xacro="http://ros.org/wiki/xacro">
+  <xacro:macro name="wheel" params="side radius width pos_x pos_y pos_z mass">
+    <link name="${side}_wheel_link">
+      <visual>
+        <origin xyz="0 0 0" rpy="${pi/2} 0 0" />
+        <geometry>
+          <cylinder radius="${radius}" length="${width}" />
+        </geometry>
+        <material name="wheel_material" />
+      </visual>
+      <collision>
+        <origin xyz="0 0 0" rpy="${pi/2} 0 0" />
+        <geometry>
+          <cylinder radius="${radius}" length="${width}" />
+        </geometry>
+      </collision>
+      <inertial>
+        <origin xyz="0 0 0" rpy="0 0 0" />
+        <mass value="${mass}" />
+        <inertia ixx="${(2/5) * mass * (radius * radius)}" ixy="0" ixz="0"
+          iyy="${(2/5) * mass * (radius * radius)}" iyz="0"
+          izz="${(2/5) * mass * (radius * radius)}" />
+      </inertial>
+    </link>
+    <gazebo reference="${side}_wheel_link">
+      <visual>
+        <material>
+          <ambient>0.1764 0.4588 0.8509 1.0</ambient>
+          <diffuse>0.1764 0.4588 0.8509 1.0</diffuse>
+          <specular>0.1764 0.4588 0.8509 1.0</specular>
+          <emissive>0.0 0.0 0.0 0.0</emissive>
+        </material>
+      </visual>
+    </gazebo>
+    <joint name="${side}_wheel_joint" type="continuous">
+      <axis xyz="0 1 0" />
+      <parent link="base_link" />
+      <child link="${side}_wheel_link" />
+      <origin xyz="${pos_x} ${pos_y} ${pos_z}" rpy="0 0 0" />
+    </joint>
+  </xacro:macro>
 </robot>

Commit message: Fix for gazebo color

File: s_description/urdf/base.urdf.xacro (robot description, xacro)
@@ -55,6 +55,6 @@
     </link>
     <gazebo reference="base_link">
-        <material name="aluminum_frame">
-            <color rgba="0.516 0.527 0.535 1" />
+        <material>
+            Gazebo/Grey
         </material>
     </gazebo>
@@ -92,5 +92,6 @@
     />
     <xacro:ld06 lidar_prefix="right_rear">
-        <origin xyz="${-(body_length / 2) - 0.030}  -${((body_width / 2) - 0)} 0.200" rpy="0 0 ${M_PI}" />
+        <origin xyz="${-(body_length / 2) - 0.030}  -${((body_width / 2) - 0)} 0.200"
+            rpy="0 0 ${M_PI}" />
     </xacro:ld06>
     <xacro:ld06 lidar_prefix="left_front">

Commit message: ld06.urdf.xacro: remove base_to_lidar_frame_${lidar_prefix} -- put this base.urdf.xacro if needed.
base.urdf.xacro: remove two lidars and replace with one.

single_lidar.launch.py: new file for single lidar launch.

base.launch.py: bring up only one lidar.

map.launch: small fixes.

slam.yaml: small tuning changes.

File: s_description/urdf/base.urdf.xacro (robot description, xacro)
@@ -91,5 +91,19 @@
         mass="0.01"
     />
-    <xacro:ld06 lidar_prefix="right_rear">
+    <link name="scan" />
+    <joint name="base_to_scan" type="fixed">
+      <parent link="base_link" />
+      <child link="scan" />
+      <origin xyz="-0.035  -0.070 0.430" rpy="0 0 ${M_PI}" />
+    </joint>
+    <xacro:ld06 lidar_prefix="top_lidar">
+        <origin xyz="0 0 0" rpy="0 0 0" />
+    </xacro:ld06>
+    <joint name="base_to_lidar_frame_top_lidar" type="fixed">
+      <parent link="scan" />
+      <child link="lidar_frame_top_lidar" />
+      <origin xyz="0 0 0" rpy="0 0 0" />
+    </joint>
+    <!-- <xacro:ld06 lidar_prefix="right_rear">
         <origin xyz="${-(body_length / 2) - 0.030}  -${((body_width / 2) - 0)} 0.200"
             rpy="0 0 ${M_PI}" />
@@ -97,5 +111,5 @@
     <xacro:ld06 lidar_prefix="left_front">
         <origin xyz="${(body_length / 2) + 0.030}  ${((body_width / 2) - 0.0)} 0.040" rpy="0 0 0" />
-    </xacro:ld06>
+    </xacro:ld06> -->
     <xacro:include filename="$(find s_description)/urdf/time_of_flight.urdf.xacro" />
     <xacro:include filename="$(find s_description)/urdf/sonar.urdf.xacro" />

File: s_description/urdf/ld06.urdf.xacro (robot description, xacro)
@@ -131,9 +131,9 @@
       <axis xyz="0 0 0" />
     </joint>
-    <joint name="base_to_lidar_frame_${lidar_prefix}" type="fixed">
+    <!-- <joint name="base_to_lidar_frame_${lidar_prefix}" type="fixed">
       <parent link="base_link" />
       <child link="lidar_frame_${lidar_prefix}" />
       <xacro:insert_block name="joint_pose" />
-    </joint>
+    </joint> -->
     <gazebo reference="lidar_frame_${lidar_prefix}">
       <sensor name="sensor_ray_${lidar_prefix}" type="ray">

Commit message: Fix for base_link collision origin

File: s_description/urdf/base.urdf.xacro (robot description, xacro)
@@ -33,5 +33,6 @@
                 <box size="${body_length} ${body_width} ${body_height}" />
             </geometry>
-            <origin rpy="0 0 0" xyz="0 0 ${(body_height/2)}" />
+            <origin rpy="0 0 0"
+                xyz="${(-body_length/2)+wheel_offset_from_front} 0 ${(body_height/2)}" />
         </collision>
         <visual>

Commit message: Fine tuning LIDAR position

File: s_description/urdf/base.urdf.xacro (robot description, xacro)
@@ -96,5 +96,5 @@
       <parent link="base_link" />
       <child link="scan" />
-      <origin xyz="-0.035  -0.070 0.430" rpy="0 0 ${M_PI}" />
+      <origin xyz="-0.018  -0.090 0.430" rpy="0 0 ${M_PI}" />
     </joint>
     <xacro:ld06 lidar_prefix="top_lidar">

Commit message: For OAK-D cameras

File: s_description/urdf/base.urdf.xacro (robot description, xacro)
@@ -143,5 +143,5 @@
         cam_yaw="-0.523599"
     /> -->
-    <!-- <xacro:oakd_link mount_point="right" />
+    <xacro:oakd_link mount_point="right" />
     <xacro:oakd_joint mount_point="right">
         <origin xyz="0.170 -0.055 0.350" rpy="0 0 -0.523599" />
@@ -162,4 +162,4 @@
         <child link="oakd_right_right_camera_optical_frame"/>
         <origin xyz="0 0 0" rpy="0 0 0" />
-    </joint> -->
+    </joint>
 </robot>
