Commit message: Trying to fix OAK-D rotation. Still not right.

File: s_description/urdf/base.urdf.xacro (robot description, xacro)
@@ -155,5 +155,5 @@
     <xacro:oakd_link mount_point="left" />
     <xacro:oakd_joint mount_point="left">
-        <origin xyz="0.170 0.055 0.350" rpy="0 0 0.523599" />
+        <origin xyz="0.170 0.055 0.350" rpy="0 0 0.5" />
     </xacro:oakd_joint>
     <link name="oakd_right_right_camera_optical_frame" />
